Commit message: Implementacion del diseño del robot final - Aun sin implementar rviz y gazebo

File: rov_description/urdf/loco.urdf.xacro (robot description, xacro)
@@ -21,5 +21,5 @@
       <!--<origin xyz=".383 -0.172 -0.0705" rpy="${pi/2} 0 ${pi}" />-->.0175
       <geometry>
-        <mesh filename="package://rov_description/meshes/LoCO_Shell.STL" scale="1 1 1" />
+        <mesh filename="package://rov_description/meshes/Rov_Max.stl" scale="1 1 1" />
       </geometry>
       <material name="Gray"/>
