Commit message: Perfeccionamiento de la ubicacion central de los propulsores

File: rov_description/urdf/rov_max.urdf.xacro (robot description, xacro)
@@ -89,19 +89,7 @@
     </inertial>
     <visual>
-      <origin xyz="0.03 0 0" rpy="${-pi/4} 0 0"/>
+      <origin xyz="0 0 0" rpy="${pi/2} 0 0"/>
       <geometry>
-        <box size="${blade_geometry}"/>
-      </geometry>
-      <material name="Green"/>
-    </visual>
-    <collision>
-      <geometry>
-        <box size="${blade_geometry}"/>
-      </geometry>
-    </collision>
-    <visual>
-      <origin xyz="-0.03 0 0" rpy="${pi/4} 0 0"/>
-      <geometry>
-        <box size="${blade_geometry}"/>
+        <mesh filename="package://rov_description/models/rov_max/meshes/t200-cw-prop.dae" scale="6 6 6"/>
       </geometry>
       <material name="Green"/>
@@ -117,5 +105,5 @@
     <child link="vert_thrust_left"/>
     <axis xyz="0 0 1"/>
-    <origin xyz="1.08 0.69949 0"/>
+    <origin xyz="1.08 0.71 0"/>
   </joint>
   <link name="vert_thrust_right">
@@ -126,19 +114,7 @@
     </inertial>
     <visual>
-      <origin xyz="0.03 0 0" rpy="${-pi/4} 0 0"/>
+      <origin xyz="0 0 0" rpy="${-pi/2} 0 0"/>
       <geometry>
-        <box size="${blade_geometry}"/>
-      </geometry>
-      <material name="Green"/>
-    </visual>
-    <collision>
-      <geometry>
-        <box size="${blade_geometry}"/>
-      </geometry>
-    </collision>
-    <visual>
-      <origin xyz="-0.03 0 0" rpy="${pi/4} 0 0"/>
-      <geometry>
-        <box size="${blade_geometry}"/>
+        <mesh filename="package://rov_description/models/rov_max/meshes/t200-ccw-prop.dae" scale="6 6 6"/>
       </geometry>
       <material name="Green"/>
@@ -154,5 +130,5 @@
     <child link="vert_thrust_right"/>
     <axis xyz="0 0 1"/>
-    <origin xyz="1.08 -0.69949 0"/>
+    <origin xyz="1.08 -0.71 0"/>
   </joint>
   <link name="left_thruster">
@@ -163,19 +139,7 @@
     </inertial>
     <visual>
-      <origin xyz="0.03 0 0" rpy="${pi/4} 0 0"/>
+      <origin xyz="0 0 0" rpy="${pi/2} 0 0"/>
       <geometry>
-        <box size="${blade_geometry}"/>
-      </geometry>
-      <material name="Green"/>
-    </visual>
-    <collision>
-      <geometry>
-        <box size="${blade_geometry}"/>
-      </geometry>
-    </collision>
-    <visual>
-      <origin xyz="-0.03 0 0" rpy="${-pi/4} 0 0"/>
-      <geometry>
-        <box size="${blade_geometry}"/>
+        <mesh filename="package://rov_description/models/rov_max/meshes/t200-ccw-prop.dae" scale="6 6 6"/>
       </geometry>
       <material name="Green"/>
@@ -191,5 +155,5 @@
     <child link="left_thruster"/>
     <axis xyz="0 0 1"/>
-    <origin xyz="-1.2429 0.69949 0" rpy="0 ${pi/2} 0"/>
+    <origin xyz="-1.2429 0.75 0" rpy="0 ${pi/2} 0"/>
     <!--In actual model: <origin xyz="-0.302 0.109 -0.000635" rpy="0 ${pi/2} 0"/> -->
   </joint>
@@ -201,19 +165,7 @@
     </inertial>
     <visual>
-      <origin xyz="0.03 0 0" rpy="${-pi/4} 0 0"/>
+      <origin xyz="0 0 0" rpy="${pi/2} 0 0"/>
       <geometry>
-        <box size="${blade_geometry}"/>
-      </geometry>
-      <material name="Green"/>
-    </visual>
-    <collision>
-      <geometry>
-        <box size="${blade_geometry}"/>
-      </geometry>
-    </collision>
-    <visual>
-      <origin xyz="-0.03 0 0" rpy="${pi/4} 0 0"/>
-      <geometry>
-        <box size="${blade_geometry}"/>
+        <mesh filename="package://rov_description/models/rov_max/meshes/t200-cw-prop.dae" scale="6 6 6"/>
       </geometry>
       <material name="Green"/>
@@ -229,5 +181,5 @@
     <child link="right_thruster"/>
     <axis xyz="0 0 1"/>
-    <origin xyz="-1.2429 -0.69949 0" rpy="0 ${pi/2} 0"/>
+    <origin xyz="-1.2429 -0.75 0" rpy="0 ${pi/2} 0"/>
     <!--In actual model: <origin xyz="-0.302 -0.109 -0.000635" rpy="0 ${pi/2} 0"/> -->
   </joint>

Commit message: Correccion de problema - Filename en rviz

File: rov_description/urdf/rov_max.urdf.xacro (robot description, xacro)
@@ -38,5 +38,5 @@
         .0175
       <geometry>
-        <mesh filename="package://rov_description/meshes/Rov_Max.stl" scale="0.01 0.01 0.01"/>
+        <mesh filename="package://rov_description/models/rov_max/meshes/rov_max.stl" scale="0.01 0.01 0.01"/>
       </geometry>
       <material name="MediumYellow"/>
