Commit message: Mejora en xacro aunque no se use

File: rov_description/urdf/rov_max.xacro (robot description, xacro)
@@ -44,20 +44,21 @@
     <visual>
       <!--The origin shift visually shifts the model to CAD model origin-->
-      <origin xyz="1.5571 0.0016 0.0084" rpy="0 0 ${pi}" />
-        .0175
-      <geometry>
-        <mesh filename="package://rov_description/models/rov_max/meshes/rov_max.stl" scale="0.01 0.01 0.01"/>
+      <origin xyz="0.15571 0.00016 0.00084" rpy="${pi} ${pi} 0" />
+      <geometry>
+        <mesh filename="package://rov_description/models/rov_max/meshes/rov_max.stl" scale="0.001 0.001 0.001"/>
       </geometry>
       <material name="MediumYellow"/>
     </visual>
     <collision>
+      <origin xyz="0.15571 0.00016 0.00084" rpy="${pi} ${pi} 0" />
       <geometry>
 	      <!--Bounding box for collision geometry used to decrease computational requirements.-->
-        <box size="3.65 2.5 1"/>
+        <box size="0.53 0.32 0.033"/>
       </geometry>
     </collision>
     <inertial>
-      <mass value="13.2"/>
-      <inertia ixx=".15" ixy="0.0" ixz="0.0" iyy=".66" iyz="0.0" izz=".53"/>
+      <origin xyz="0.15571 0.00016 0.00084" rpy="${pi} ${pi} 0" />
+      <mass value="4.488"/>
+      <inertia ixx=".03870488600000001" ixy="0.0" ixz="0.0" iyy=".067961036" iyz="0.0" izz=".10585135000000001"/>
     </inertial>
   </link>
@@ -65,5 +66,6 @@
     <parent link="rov_max_frame"/>
     <child link="rov_max_shell"/>
-    <origin xyz="0 0 0"/>
+    <origin xyz="0.15571 0.00016 0.00084" rpy="${pi} ${pi} 0"/>
+    <axis xyz="0 0 1"/>
   </joint>
   <!-- ***************************** -->
@@ -71,20 +73,13 @@
   <!-- ***************************** -->
   <link name="camera">
-    <origin xyz="0 0 0" rpy="0 0 0"/>
-    <visual>
-      <origin xyz="0.025223 0 0" rpy="0 0 0"/>
-      <geometry>
-        <box size="0.2 0.4 0.2"/>
+    <visual>
+      <geometry>
+        <box size="0.02 0.04 0.02"/>
       </geometry>
       <material name="Gray"/>
     </visual>
-    <collision>
-      <geometry>
-        <box size="0.2 0.4 0.2"/>
-      </geometry>
-    </collision>
-    <inertial>
-      <mass value="${negligible}"/>
-      <inertia ixx="${negligible}" ixy="0.00" ixz="0.00" iyy="${negligible}" iyz="0.00" izz="${negligible}"/>
+    <inertial>
+      <mass value="0.00133"/>
+      <inertia ixx="0.001" ixy="0.00" ixz="0.00" iyy="0.001" iyz="0.00" izz="0.001"/>
     </inertial>
   </link>
@@ -92,5 +87,6 @@
     <parent link="rov_max_shell"/>
     <child link="camera"/>
-    <origin xyz="1.5571 0 0"/>
+    <origin xyz="0.15571 0 0"/>
+    <axis xyz="0 0 1"/>
   </joint>
   <!-- ***************************** -->
@@ -100,104 +96,83 @@
     <origin xyz="0 0 0" rpy="0 0 0"/>
     <inertial>
-      <mass value="${negligible}"/>
-      <inertia ixx="${negligible}" ixy="0.00" ixz="0.00" iyy="${negligible}" iyz="0.00" izz="${negligible}"/>
+      <mass value="0.001"/>
+      <inertia ixx="0.001" ixy="0.00" ixz="0.00" iyy="0.001" iyz="0.00" izz="0.001"/>
+    </inertial>
+    <visual>
+      <origin xyz="0 0 0" rpy="${-pi/2} 0 0"/>
+      <geometry>
+        <mesh filename="package://rov_description/models/rov_max/meshes/t200-ccw-prop.dae" scale="0.8 0.8 0.8"/>
+      </geometry>
+      <material name="Green"/>
+    </visual>
+  </link>
+  <joint name="shell_to_vert_thrust_left" type="continuous">
+    <parent link="rov_max_shell"/>
+    <child link="vert_thrust_left"/>
+    <axis xyz="0 0 1"/>
+    <origin xyz="0.108 0.071 0" rpy="0 0 0"/>
+  </joint>
+  <!-- ***************************** -->
+  <!-- *** VERTICAL THRUST RIGHT *** -->
+  <!-- ***************************** -->
+  <link name="vert_thrust_right">
+    <origin xyz="0 0 0" rpy="0 0 0"/>
+    <inertial>
+      <mass value="0.001"/>
+      <inertia ixx="0.001" ixy="0.00" ixz="0.00" iyy="0.001" iyz="0.00" izz="0.001"/>
     </inertial>
     <visual>
       <origin xyz="0 0 0" rpy="${pi/2} 0 0"/>
       <geometry>
-        <mesh filename="package://rov_description/models/rov_max/meshes/t200-cw-prop.dae" scale="6 6 6"/>
-      </geometry>
-      <material name="Green"/>
-    </visual>
-    <collision>
-      <geometry>
-        <box size="${blade_geometry}"/>
-      </geometry>
-    </collision>
-  </link>
-  <joint name="shell_to_vert_thrust_left" type="continuous">
-    <parent link="rov_max_shell"/>
-    <child link="vert_thrust_left"/>
-    <axis xyz="0 0 1"/>
-    <origin xyz="1.08 0.71 0"/>
-  </joint>
-  <!-- ***************************** -->
-  <!-- *** VERTICAL THRUST RIGHT *** -->
-  <!-- ***************************** -->
-  <link name="vert_thrust_right">
-    <origin xyz="0 0 0" rpy="0 0 0"/>
-    <inertial>
-      <mass value="${negligible}"/>
-      <inertia ixx="${negligible}" ixy="0.00" ixz="0.00" iyy="${negligible}" iyz="0.00" izz="${negligible}"/>
+        <mesh filename="package://rov_description/models/rov_max/meshes/t200-cw-prop.dae" scale="0.8 0.8 0.8"/>
+      </geometry>
+      <material name="Green"/>
+    </visual>
+  </link>
+  <joint name="shell_to_vert_thrust_right" type="continuous">
+    <parent link="rov_max_shell"/>
+    <child link="vert_thrust_right"/>
+    <axis xyz="0 0 1"/>
+    <origin xyz="0.108 -0.071 0"/>
+  </joint>
+  <!-- ***************************** -->
+  <!-- ******* THRUSTER LEFT ******* -->
+  <!-- ***************************** -->
+  <link name="left_thruster">
+    <origin xyz="0 0 0" rpy="0 0 0"/>
+    <inertial>
+      <mass value="0.001"/>
+      <inertia ixx="0.001" ixy="0.00" ixz="0.00" iyy="0.001" iyz="0.00" izz="0.001"/>
     </inertial>
     <visual>
       <origin xyz="0 0 0" rpy="${-pi/2} 0 0"/>
       <geometry>
-        <mesh filename="package://rov_description/models/rov_max/meshes/t200-ccw-prop.dae" scale="6 6 6"/>
-      </geometry>
-      <material name="Green"/>
-    </visual>
-    <collision>
-      <geometry>
-        <box size="${blade_geometry}"/>
-      </geometry>
-    </collision>
-  </link>
-  <joint name="shell_to_vert_thrust_right" type="continuous">
-    <parent link="rov_max_shell"/>
-    <child link="vert_thrust_right"/>
-    <axis xyz="0 0 1"/>
-    <origin xyz="1.08 -0.71 0"/>
-  </joint>
-  <!-- ***************************** -->
-  <!-- ******* THRUSTER LEFT ******* -->
-  <!-- ***************************** -->
-  <link name="left_thruster">
-    <origin xyz="0 0 0" rpy="0 0 0"/>
-    <inertial>
-      <mass value="${negligible}"/>
-      <inertia ixx="${negligible}" ixy="0.00" ixz="0.00" iyy="${negligible}" iyz="0.00" izz="${negligible}"/>
+        <mesh filename="package://rov_description/models/rov_max/meshes/t200-ccw-prop.dae" scale="0.8 0.8 0.8"/>
+      </geometry>
+      <material name="Green"/>
+    </visual>
+  </link>
+  <joint name="shell_to_left_thrust" type="continuous">
+    <parent link="rov_max_shell"/>
+    <child link="left_thruster"/>
+    <axis xyz="0 0 1"/>
+    <origin xyz="-0.12429 0.075 0" rpy="0 ${pi/2} 0"/>
+  </joint>
+  <!-- ***************************** -->
+  <!-- ******* THRUSTER RIGHT ****** -->
+  <!-- ***************************** -->
+  <link name="right_thruster">
+    <origin xyz="0 0 0" rpy="0 0 0"/>
+    <inertial>
+      <mass value="0.001"/>
+      <inertia ixx="0.001" ixy="0.00" ixz="0.00" iyy="0.001" iyz="0.00" izz="0.001"/>
     </inertial>
     <visual>
       <origin xyz="0 0 0" rpy="${pi/2} 0 0"/>
       <geometry>
-        <mesh filename="package://rov_description/models/rov_max/meshes/t200-ccw-prop.dae" scale="6 6 6"/>
-      </geometry>
-      <material name="Green"/>
-    </visual>
-    <collision>
-      <geometry>
-        <box size="${blade_geometry}"/>
-      </geometry>
-    </collision>
-  </link>
-  <joint name="shell_to_left_thrust" type="continuous">
-    <parent link="rov_max_shell"/>
-    <child link="left_thruster"/>
-    <axis xyz="0 0 1"/>
-    <origin xyz="-1.2429 0.75 0" rpy="0 ${pi/2} 0"/>
-    <!--In actual model: <origin xyz="-0.302 0.109 -0.000635" rpy="0 ${pi/2} 0"/> -->
-  </joint>
-  <!-- ***************************** -->
-  <!-- ******* THRUSTER RIGHT ****** -->
-  <!-- ***************************** -->
-  <link name="right_thruster">
-    <origin xyz="0 0 0" rpy="0 0 0"/>
-    <inertial>
-      <mass value="${negligible}"/>
-      <inertia ixx="${negligible}" ixy="0.00" ixz="0.00" iyy="${negligible}" iyz="0.00" izz="${negligible}"/>
-    </inertial>
-    <visual>
-      <origin xyz="0 0 0" rpy="${pi/2} 0 0"/>
-      <geometry>
-        <mesh filename="package://rov_description/models/rov_max/meshes/t200-cw-prop.dae" scale="6 6 6"/>
-      </geometry>
-      <material name="Green"/>
-    </visual>
-    <collision>
-      <geometry>
-        <box size="${blade_geometry}"/>
-      </geometry>
-    </collision>
+        <mesh filename="package://rov_description/models/rov_max/meshes/t200-cw-prop.dae" scale="0.8 0.8 0.8"/>
+      </geometry>
+      <material name="Green"/>
+    </visual>
   </link>
   <joint name="shell_to_right_thrust" type="continuous">
@@ -205,6 +180,28 @@
     <child link="right_thruster"/>
     <axis xyz="0 0 1"/>
-    <origin xyz="-1.2429 -0.75 0" rpy="0 ${pi/2} 0"/>
-    <!--In actual model: <origin xyz="-0.302 -0.109 -0.000635" rpy="0 ${pi/2} 0"/> -->
+    <origin xyz="-0.12429 -0.075 0" rpy="0 ${pi/2} 0"/>
+  </joint>
+  <!-- ***************************** -->
+  <!-- ******* THRUSTER CENTR ****** -->
+  <!-- ***************************** -->
+  <link name="center_thruster">
+    <origin xyz="0 0 0" rpy="0 0 0"/>
+    <inertial>
+      <mass value="0.001"/>
+      <inertia ixx="0.001" ixy="0.00" ixz="0.00" iyy="0.001" iyz="0.00" izz="0.001"/>
+    </inertial>
+    <visual>
+      <origin xyz="0 0 0" rpy="${-pi/2} 0 0"/>
+      <geometry>
+        <mesh filename="package://rov_description/models/rov_max/meshes/t200-ccw-prop.dae" scale="0.8 0.8 0.8"/>
+      </geometry>
+      <material name="Green"/>
+    </visual>
+  </link>
+  <joint name="shell_to_center_thrust" type="continuous">
+    <parent link="rov_max_shell"/>
+    <child link="center_thruster"/>
+    <axis xyz="0 0 1"/>
+    <origin xyz="-0.175 -0.0 0" rpy="0 0 0"/>
   </joint>
 </robot>

Commit message: Ordenar pkgs para diferentes acciones generales

File: rov_description/urdf/rov_max.xacro (robot description, xacro)
@@ -46,5 +46,5 @@
       <origin xyz="0.15571 0.00016 0.00084" rpy="${pi} ${pi} 0" />
       <geometry>
-        <mesh filename="package://rov_description/models/rov_max/meshes/rov_max.stl" scale="0.001 0.001 0.001"/>
+        <mesh filename="package://rov_gazebo/models/rov_max/meshes/rov_max.stl" scale="0.001 0.001 0.001"/>
       </geometry>
       <material name="MediumYellow"/>
@@ -102,5 +102,5 @@
       <origin xyz="0 0 0" rpy="${-pi/2} 0 0"/>
       <geometry>
-        <mesh filename="package://rov_description/models/rov_max/meshes/t200-ccw-prop.dae" scale="0.8 0.8 0.8"/>
+        <mesh filename="package://rov_gazebo/models/rov_max/meshes/t200-ccw-prop.dae" scale="0.8 0.8 0.8"/>
       </geometry>
       <material name="Green"/>
@@ -125,5 +125,5 @@
       <origin xyz="0 0 0" rpy="${pi/2} 0 0"/>
       <geometry>
-        <mesh filename="package://rov_description/models/rov_max/meshes/t200-cw-prop.dae" scale="0.8 0.8 0.8"/>
+        <mesh filename="package://rov_gazebo/models/rov_max/meshes/t200-cw-prop.dae" scale="0.8 0.8 0.8"/>
       </geometry>
       <material name="Green"/>
@@ -148,5 +148,5 @@
       <origin xyz="0 0 0" rpy="${-pi/2} 0 0"/>
       <geometry>
-        <mesh filename="package://rov_description/models/rov_max/meshes/t200-ccw-prop.dae" scale="0.8 0.8 0.8"/>
+        <mesh filename="package://rov_gazebo/models/rov_max/meshes/t200-ccw-prop.dae" scale="0.8 0.8 0.8"/>
       </geometry>
       <material name="Green"/>
@@ -171,5 +171,5 @@
       <origin xyz="0 0 0" rpy="${pi/2} 0 0"/>
       <geometry>
-        <mesh filename="package://rov_description/models/rov_max/meshes/t200-cw-prop.dae" scale="0.8 0.8 0.8"/>
+        <mesh filename="package://rov_gazebo/models/rov_max/meshes/t200-cw-prop.dae" scale="0.8 0.8 0.8"/>
       </geometry>
       <material name="Green"/>
@@ -194,5 +194,5 @@
       <origin xyz="0 0 0" rpy="${-pi/2} 0 0"/>
       <geometry>
-        <mesh filename="package://rov_description/models/rov_max/meshes/t200-ccw-prop.dae" scale="0.8 0.8 0.8"/>
+        <mesh filename="package://rov_gazebo/models/rov_max/meshes/t200-ccw-prop.dae" scale="0.8 0.8 0.8"/>
       </geometry>
       <material name="Green"/>

Commit message: Añadir sonar a rviz2

File: rov_description/urdf/rov_max.xacro (robot description, xacro)
@@ -91,4 +91,25 @@
   </joint>
   <!-- ***************************** -->
+  <!-- ********** SONAR ************ -->
+  <!-- ***************************** -->
+  <link name="sonar_link">
+    <visual>
+      <geometry>
+        <box size="0.01 0.02 0.01"/>
+      </geometry>
+      <material name="Gray"/>
+    </visual>
+    <inertial>
+      <mass value="0.002667"/>
+      <inertia ixx="0.001" ixy="0.00" ixz="0.00" iyy="0.001" iyz="0.00" izz="0.001"/>
+    </inertial>
+  </link>
+  <joint name="shell_to_sonar" type="fixed">
+    <parent link="rov_max_shell"/>
+    <child link="sonar_link"/>
+    <origin xyz="0.075 0 0.05"/>
+    <axis xyz="0 0 1"/>
+  </joint>
+  <!-- ***************************** -->
   <!-- **** VERTICAL THRUST LEFT *** -->
   <!-- ***************************** -->
