Commit message: Xacro corregido

File: auv_max_description/urdf/auv_max.xacro (robot description, xacro)
@@ -66,5 +66,5 @@
     <parent link="auv_max_frame"/>
     <child link="auv_max_shell"/>
-    <origin xyz="0.15571 0.00016 0.00084" rpy="${pi} ${pi} 0"/>
+    <origin xyz="0.15571 0.00016 0.00084" rpy="${pi} ${pi} ${-pi}"/>
     <axis xyz="0 0 1"/>
   </joint>
@@ -80,6 +80,6 @@
     </visual>
     <inertial>
-      <mass value="0.00133"/>
-      <inertia ixx="0.001" ixy="0.00" ixz="0.00" iyy="0.001" iyz="0.00" izz="0.001"/>
+      <mass value="0.002"/>
+      <inertia ixx="1.11e-7" ixy="0.00" ixz="0.00" iyy="4.45e-8" iyz="0.00" izz="1.11e-7"/>
     </inertial>
   </link>
@@ -101,6 +101,6 @@
     </visual>
     <inertial>
-      <mass value="0.002667"/>
-      <inertia ixx="0.001" ixy="0.00" ixz="0.00" iyy="0.001" iyz="0.00" izz="0.001"/>
+      <mass value="0.00097"/>
+      <inertia ixx="1.11e-7" ixy="0.00" ixz="0.00" iyy="4.45e-8" iyz="0.00" izz="1.11e-7"/>
     </inertial>
   </link>
@@ -117,5 +117,5 @@
     <origin xyz="0 0 0" rpy="0 0 0"/>
     <inertial>
-      <mass value="0.001"/>
+      <mass value="0.002"/>
       <inertia ixx="0.001" ixy="0.00" ixz="0.00" iyy="0.001" iyz="0.00" izz="0.001"/>
     </inertial>
@@ -140,5 +140,5 @@
     <origin xyz="0 0 0" rpy="0 0 0"/>
     <inertial>
-      <mass value="0.001"/>
+      <mass value="0.002"/>
       <inertia ixx="0.001" ixy="0.00" ixz="0.00" iyy="0.001" iyz="0.00" izz="0.001"/>
     </inertial>
@@ -163,5 +163,5 @@
     <origin xyz="0 0 0" rpy="0 0 0"/>
     <inertial>
-      <mass value="0.001"/>
+      <mass value="0.002"/>
       <inertia ixx="0.001" ixy="0.00" ixz="0.00" iyy="0.001" iyz="0.00" izz="0.001"/>
     </inertial>
@@ -186,5 +186,5 @@
     <origin xyz="0 0 0" rpy="0 0 0"/>
     <inertial>
-      <mass value="0.001"/>
+      <mass value="0.002"/>
       <inertia ixx="0.001" ixy="0.00" ixz="0.00" iyy="0.001" iyz="0.00" izz="0.001"/>
     </inertial>
@@ -209,5 +209,5 @@
     <origin xyz="0 0 0" rpy="0 0 0"/>
     <inertial>
-      <mass value="0.001"/>
+      <mass value="0.002"/>
       <inertia ixx="0.001" ixy="0.00" ixz="0.00" iyy="0.001" iyz="0.00" izz="0.001"/>
     </inertial>
